File: eagle/printed/202403-controller-rev2.sch (EAGLE design)
At the start: 54 parts, among them J2 1-770166-0, J3 1-794073-0, J4 JST-XH-04-PIN-ROUND-PAD, Q1 200mA/40V, Q2 20V/4.2A/52mΩ/1.4W, U1 AP63205WU-7, U2 TJA1055T_3_2Z, U3 MIC5504-3.3YM5-TR, U4 ESP32-S3-WROOM-1-N16R2, U5 VO2223B-X007T, U6 TCMT1106, U7 TCMT1106, U8 BME280

Commit message: Remove old eagle files now that we have git history
Parts:
- removed DL, HV, SP, TACH, VCC: PTR1B1,27, testpad:PTR1B1,27
- removed H2: MOUNT-HOLE3.3, holes:MOUNT-HOLE3.3
- removed J3: 1-794073-0, Terminals and sockets:1-794073-0
- removed Q1: 200mA/40V, SparkFun-DiscreteSemi:TRANS_PNP-PMBT3906|MMBT3906L
- removed Q2: 20V/4.2A/52mΩ/1.4W, SparkFun-DiscreteSemi:MOSFET_PCH-DMG2305UX-7
- removed R13, R14, R9: 4.7k, SparkFun-Resistors:4.7KOHM-0603-1/10W-1%
- removed R17, R8: 47k, SparkFun-Resistors:47KOHM-0603-1/10W-1%
- removed R2: 510, Resistors:510OHM-0603-1/10W-5%
- removed R3: 2.2k, SparkFun-Resistors:2.2KOHM-0603-1/10W-1%
- removed R4: 100, Resistors:100OHM-0805-1/10W-5%-400V
- removed R5: 220, SparkFun-Resistors:220OHM-0603-1/10W-1%
- removed U3: MIC5504-3.3YM5-TR, MIC5504-3.3YM5-TR:MIC5504-3.3YM5-TR
- added B1: BAT-HLD-012-SMT, Battery holders:BAT-HLD-012-SMT
- added BOOT: PTR1B1,27, testpad:PTR1B1,27
- added C12: 0.1uF, SparkFun-Capacitors:0.1UF-0603-25V-5%
- added D2: 1A/23V/620mV, SparkFun-DiscreteSemi:DIODE-SCHOTTKY-BAT20J
- added JP1: JUMPER-SMT_2_NC_TRACE_NO-SILK, SparkFun-Jumpers:JUMPER-SMT_2_NC_TRACE_NO-SILK
- added JP2, RST: JUMPER-SMT_2_NO_NO-SILK, SparkFun-Jumpers:JUMPER-SMT_2_NO_NO-SILK
- added R40: 120, Resistors:120OHM-0603-1/10W-5%
- added RV1, RV2: ZV35K1210251NIR1, Bourns Varistor ZV35K1210251NIR1:ZV35K1210251NIR1
- added U9: SP3485CN-L, MaxLinear RS485 SP3485CN-L:SP3485CN-L
- added X3: FFC2B35-18-G-EYE_SPI, GCT FFC2B35-18-G:FFC2B35-18-G-EYE_SPI
- C1: device SparkFun-Capacitors:10UF-1210-50V-20% -> SparkFun-Capacitors:10UF-1206-6.3V-20%
- C11: value 10nF -> 10uF; device Capacitors:10NF-0805-400V-20% -> SparkFun-Capacitors:10UF-1206-6.3V-20%
- C8: value 10nF -> 1.0uF; device SparkFun-Capacitors:10NF-0603-50V-10% -> SparkFun-Capacitors:1.0UF-0603-16V-10%
- C9: value 1.0uF -> 0.1uF; device SparkFun-Capacitors:1.0UF-0603-16V-10% -> SparkFun-Capacitors:0.1UF-0603-25V-5%
- J2: value 1-770166-0 -> 282834-3; device Terminals and sockets:1-770166-0 -> TE terminal block 282834-3:282834-3
- L1: value 4.7μH -> 4.7μH_SHIELDED_INDUCTOR; device SparkFun-Coils:4.7μH_SHIELDED_INDUCTORNPIS_LS -> SparkFun-Coils:4.7μH_SHIELDED_INDUCTOR
- R1: value 510 -> 1k; device Resistors:510OHM-0603-1/10W-5% -> SparkFun-Resistors:1KOHM-0603-1/10W-1%
- R10: value 120 -> 220; device Resistors:120OHM-0603-1/10W-5% -> SparkFun-Resistors:220OHM-0603-1/10W-1%
- R11, R7: value 4.7k -> 1k; device SparkFun-Resistors:4.7KOHM-0603-1/10W-1% -> SparkFun-Resistors:1KOHM-0603-1/10W-1%
- R6: value 2.2k -> 220; device SparkFun-Resistors:2.2KOHM-0603-1/10W-1% -> SparkFun-Resistors:220OHM-0603-1/10W-1%
- U1: value AP63205WU-7 -> AP63203WU-7; device Diodes buck converter:AP63205WU-7 -> Diodes buck converter:AP63203WU-7
- U2: value TJA1055T_3_2Z -> SCD-40; device TJA1055T_3_2Z:TJA1055T_3_2Z -> Adafruit SCD-41:SCD-40
- U5: value VO2223B-X007T -> G3VM-61VY3_TR_; device VO2223B-X007T:VO2223B-X007T -> Omron SSR G3VM-61VY3_TR_:G3VM-61VY3_TR_
- U6: value TCMT1106 -> G3VM-61VY3_TR_; device TCMT1106:TCMT1106 -> Omron SSR G3VM-61VY3_TR_:G3VM-61VY3_TR_
- U7: value TCMT1106 -> RX8111CE_B0; device TCMT1106:TCMT1106 -> RX8111CE_B0:RX8111CE_B0
- U8: value BME280 -> STS35-DIS; device SparkFun-Sensors:BME280 -> STS35-DIS:STS35-DIS
Connections:
- removed net CANH: J4-3.S, R1.2, U2.CANH
- removed net CANL: J4-2.S, R2.2, U2.CANL
- removed net CAN_ERR: R14.1, U2.!ERR, U4.IO8
- removed net CAN_RX: R13.1, U2.RXD, U4.IO17
- removed net CAN_TX: U2.TXD, U4.IO18
- removed net HV_IO: R10.2, U4.IO35
- removed net HV_SW: HV.TP, R10.1, U5.A
- removed net LINE: C11.1, J2.1, U5.MT2
- removed net M+10V: J3.7, Q1.E, R8.2
- removed net M+15V: J3.2, R6.1
- removed net MGND: J3.6, U7.E
- removed net MSPEED: J3.3, Q1.C
- removed net MTR: J2.2, R4.1, U5.MT1
- removed net N$11: C11.2, R4.2
- removed net N$13: R5.1, U7.A
- removed net N$15: Q1.B, R8.1, R9.1
- removed net N$16: R9.2, U7.C
- removed net N$8: C8.2, R3.1, U2.!WAKE, U2.BAT
- removed net SPEED_IO: R5.2, SP.TP, U4.IO9
- removed net TACH: J3.1, U6.K
- removed net TACH_IO: TACH.TP, U4.IO13, U6.C
- removed net VCC: C3.1, C4.1, C5.1, L1.2, Q2.D, U1.FB, U2.!STB, U2.EN, U2.VCC, VCC.TP
- new net COOL_IO: R6.2, U4.IO9
- new net DC: U4.IO13, X3.DC
- new net DISP_RST: U4.IO12, X3.RESET
- new net HEAT_IO: R10.2, U4.IO3
- new net LITE: U4.IO48, X3.BACKLITE
- new net MISO: U4.IO14, X3.MISO
- new net MOSI: U4.IO21, X3.MOSI
- new net N$4: R6.1, U5.A
- new net R: J2.2, RV1.1, RV2.2, U5.D2, U6.D1
- new net RS485A: J4-2.S, R40.1, U9.B
- new net RS485B: J4-3.S, JP1.1, U9.A
- new net RS485_DE: U4.IO18, U9.!RE, U9.DE
- new net RS485_RX: U4.IO8, U9.RO
- new net RS485_TX: U4.IO17, U9.DI
- new net RTC_VBAT: R1.2, U7.VBAT
- new net RTC_VOUT: C8.2, U7.VOUT
- new net SCK: U4.IO47, X3.SCK
- new net TE: U4.IO10, X3.BUSY/TE
- new net TS_INT: U4.IO11, X3.INT
- new net W: J2.1, RV1.2, U6.D2
- new net Y: J2.3, RV2.1, U5.D1
- net 3.3V: now also C11.1, C12.2, C14.1, C3.1, C4.1, C5.2, C9.1, L1.2, U1.FB, U2.VDD, U2.VDDH, U7.VDD, U7.VIO, U9.VCC, X3.VCC; no longer C14.2, R13.2, R14.2, U3.VOUT, U8.!CS, U8.VDDIO
- net GND: now also B1.3, C11.2, C12.1, C14.2, C5.1, C9.2, JP2.2, RST.2, U6.K, U7.GND, U8.ADDR, U8.R, U8.VSS, U9.GND, X3.DISP_CS, X3.GND; no longer C14.1, C5.2, C9.1, J3.8, R17.1, U3.GND, U6.E, U7.K, U8.SDO/ADR
- net N$10: now also R10.1; no longer R6.2
- net N$3: now also BOOT.TP, JP2.1; no longer DL.TP
- net N$5: now also JP1.2, R40.2; no longer R2.1, U2.RTL
- net N$6: now also B1.1; no longer U2.RTH
- net N$9: now also RST.1
- net REG_IN: now also C1.1, D2.C, U1.EN, U1.VIN; no longer C9.2, Q2.S, U3.EN, U3.VIN
- net SCL: now also U2.SCL, U4.IO36, U7.SCL, U8.SCL, X3.SCL; no longer U4.IO39, U8.SCK/SCL
- net SDA: now also U2.SDA, U4.IO39, U7.SDA, U8.SDA, X3.SDA; no longer U4.IO36, U8.SDI/SDA
- net VIN: now also D2.A; no longer C1.1, J3.4, R3.2, U1.EN, U1.VIN
- net V_USB: no longer Q2.G, R17.2
Other:
- note added: "3.3V REGULATOR"
- note added: "8.6-10ma / 0.022W"
- note added: "RS485"
- note added: "Strapping: IO0/3/45/46"
- note removed: "16-20ma / 0.048W"
- note removed: "1uF filter on VOUT if not near other filters"
- note removed: "5V REGULATOR"
- note removed: "8.6-10.4ma / 0.024W"
- note removed: "CAN INTERFACE"
- note removed: "~6.4ma / 0.09W"
- moved on the sheet: C1, C11, C14, C2, C3, C4, C5, C8, C9, D1, J4-1, J4-2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
