File: eagle/printed/202403-zone_ctrl.brd (EAGLE design)
At the start: 78.7 x 113 mm, 95 parts, among them IC1 ATTINY426-MU, J10 1-770166-0, J11 1-770166-0, J13 FEMALE 2x3, J2 282834-8, J3 282834-8, J4 282834-8, J5 282834-8, J6 282834-8, J7 282834-8, J8 4DB-P108-04, J9 282834-2, Q2 20V/4.2A/52mΩ/1.4W, U1 AP63205WU-7, U11 LTV-844S, U12 LTV-844S, U13 LTV-844S, U14 LTV-844S, U16 CPC1966Y, U17 CPC1966Y, U2 TJA1055T_3_2Z, U3 MIC5504-3.3YM5-TR, U4 ESP32-S3-WROOM-1U-N16R8, U5 G3VM-61VY3_TR_, U6 G3VM-61VY3_TR_, U7 G3VM-61VY3_TR_, U8 G3VM-61VY3_TR_, U9 SP3485CN-L, X1 JST-XH-04-PIN-ROUND-PAD, X3 FFC2B35-18-G-EYE_SPI

Commit message: Remove old eagle files now that we have git history
Parts:
- removed C8: 10nF, SparkFun-Capacitors:0603
- removed C9: 1.0uF, SparkFun-Capacitors:0603
- removed DL, VCC: PTR1B1,27, testpad:B1,27
- removed IC1: ATTINY426-MU, ATTINY426-MU:QFN40P300X300X90-21N
- removed J10: 1-770166-0, Terminals and sockets:17701660
- removed J13: FEMALE 2x3, SparkFun-Connectors:2X3
- removed Q2: 20V/4.2A/52mΩ/1.4W, SparkFun-DiscreteSemi:SOT23-3
- removed R13, R14: 4.7k, SparkFun-Resistors:0603
- removed R17: 47k, SparkFun-Resistors:0603
- removed R3: 2.2k, SparkFun-Resistors:0603
- removed U3: MIC5504-3.3YM5-TR, MIC5504-3.3YM5-TR:SOT95P280X145-5N
- added BOOT, RST: JUMPER-SMT_2_NO_NO-SILK, SparkFun-Jumpers:SMT-JUMPER_2_NO_NO-SILK
- added BOOT_TP: PTR1B1,27, testpad:B1,27
- added D2, D3, D4, D5, D6: 1A/23V/620mV, SparkFun-DiscreteSemi:SOD-323
- added J12: 455-1750-1-ND, SparkFun-Connectors:1X03
- C1: device SparkFun-Capacitors:1210 -> SparkFun-Capacitors:1206
- J9: value 282834-2 -> 282834-3; device TE terminal block 282834-2:282834-2_1 -> Terminals and sockets:2828343
- L1: value 4.7μH -> 4.7μH_SHIELDED_INDUCTOR; device SparkFun-Coils:INDUCTOR_4X4MM -> SparkFun-Coils:1008(2520)
- R1, R2: value 510 -> 2.2k; device Resistors:0603 -> SparkFun-Resistors:0603
- R20, R21, R22, R23, R24, R25, R26, R27, R28, R29, R30, R31, R32, R33, R34, R35: value 10k -> 22k
- R7, R8: value 4.7k -> 1k
- U1: value AP63205WU-7 -> AP63203WU-7
- U2: value TJA1055T_3_2Z -> ATTINY426-MU; device TJA1055T_3_2Z:SOIC127P600X175-14N -> ATTINY426-MU:QFN40P300X300X90-21N
- X1: value JST-XH-04-PIN-ROUND-PAD -> JST-XH-02-PIN-ROUND-PAD; device Rembrandt Electronics - JST XH Connectors v1-0:JST-XH-04-PACKAGE-ROUND-PAD -> Rembrandt Electronics - JST XH Connectors v1-0:JST-XH-02-PACKAGE-ROUND-PAD
- moved C5 54.1 mm to (5.59, 50.4), turned to 90 degrees
- moved R33 53.4 mm to (15.5, 94.7), turned to 90 degrees
- moved R2 46.8 mm to (36.3, 51.1)
- moved R1 46.4 mm to (33.8, 51.1)
- moved U2 42.5 mm to (43.3, 54.5), turned to 90 degrees
- moved R8 34.5 mm to (33.8, 4.57), turned to 90 degrees
- moved R7 34.3 mm to (31.4, 4.57), turned to 90 degrees
- moved R32 22.7 mm to (12.8, 94.7), turned to 90 degrees
- moved X1 20.2 mm to (23.0, 2.41), turned to 0 degrees
- moved X3 19.4 mm to (44.6, 6.35), turned to 0 degrees
- moved C1 14.2 mm to (14.0, 13.5)
- moved FC1_V 12.7 mm to (39.8, 30.5)
- moved C4 12.5 mm to (24.0, 16.5)
- moved FC1_OB 11.7 mm to (42.8, 31.4)
- moved C2 10.9 mm to (21.5, 12.7), turned to 270 degrees
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Connections:
- removed net CANH: R1.2, U2.11, X1.3
- removed net CANL: R2.2, U2.12, X1.2
- removed net CAN_ERR: R14.1, U2.4, U4.12
- removed net CAN_RX: R13.1, U2.3, U4.10
- removed net CAN_TX: U2.2, U4.11
- removed net N$5: R2.1, U2.9
- removed net N$6: R1.1, U2.8
- removed net N$8: C8.2, R3.1, U2.14, U2.7
- removed net SD_CS: U4.21, X3.9
- removed net TS3_Y: J7.7, R34.2
- removed net TS3_Y_IO: IC1.16, U14.14
- removed net TS_CS: U4.22, X3.7
- removed net VCC: C3.1, C4.1, C5.1, L1.P$2, Q2.3, U1.1, U2.10, U2.5, U2.6, VCC.TP
- removed net VLV_SW: J2.4, J2.8, J3.4, J3.8, R32.2
- removed net VLV_SW_IO: IC1.18, U14.10
- new net DISP_RST: U4.20, X3.11
- new net TE: U4.15, X3.3
- new net VLV1/2_SW: D2.A, D5.C, R33.2
- new net VLV1/2_SW_IO: R2.1, U14.12, U2.17
- new net VLV1_SW: D2.C, J2.4
- new net VLV2_SW: D5.A, J2.8
- new net VLV3/4_SW: D3.C, D6.A, R32.2
- new net VLV3/4_SW_IO: R1.1, U14.10, U2.18
- new net VLV3_SW: D3.A, J3.4
- new net VLV4_SW: D6.C, J3.8
- net 3.3V: now also C3.1, C4.1, C5.2, J12.2, L1.2, R1.2, R2.2, U1.1, U2.4; no longer IC1.4, J13.2, R13.2, R14.2, U3.5
- net DC: now also U4.21; no longer U4.20
- net FC1_OB_IO: now also U2.2; no longer IC1.2
- net FC1_V_IO: now also U2.1; no longer IC1.1
- net FC2_OB_IO: now also U2.6; no longer IC1.6
- net FC2_V_IO: now also U2.5; no longer IC1.5
- net FC3_OB_IO: now also U2.8; no longer IC1.8
- net FC3_V_IO: now also U2.7; no longer IC1.7
- net FC4_OB_IO: now also U2.10; no longer IC1.10
- net FC4_V_IO: now also U2.9; no longer IC1.9
- net GND: now also BOOT.2, C5.1, J12.3, J9.3, RST.2, U2.21, U2.3, X1.2, X3.10; no longer C5.2, C8.1, C9.1, IC1.21, IC1.3, J10.2, J13.6, R17.1, U2.13, U3.2, X1.4
- net LITE: now also U4.25; no longer U4.15
- net MISO: now also U4.22; no longer U4.19
- net MOSI: now also U4.23; no longer U4.18
- net N$1: now also L1.1; no longer L1.P$1
- net N$3: now also BOOT.1, BOOT_TP.TP; no longer DL.TP
- net N$9: now also RST.1
- net REG_IN: now also C1.1, D4.C, U1.2, U1.3; no longer C9.2, Q2.2, U3.1, U3.3
- net SCK: now also U4.24; no longer U4.17
- net SCL: now also U4.19; no longer U4.23
- net SDA: now also U4.18; no longer U4.24
- net TS1_W_IO: now also U2.13; no longer IC1.13
- net TS1_Y_IO: now also U2.12; no longer IC1.12
- net TS2_W_IO: now also U2.11; no longer IC1.11
- net TS2_Y_IO: now also U2.14; no longer IC1.14
- net TS3_W_IO: now also U2.15; no longer IC1.15
- net TS4_W: now also R34.2; no longer R33.2
- net TS4_W_IO: now also U14.14, U2.16; no longer IC1.17, U14.12
- net TS_INT: now also U4.17; no longer U4.25
- net UART: now also U2.20; no longer IC1.20
- net UPDI: now also J12.1, U2.19; no longer IC1.19, J13.1
- net VIN: now also D4.A; no longer C1.1, J10.1, R3.2, U1.2, U1.3
- net V_USB: no longer Q2.1, R17.2
Routing:
- net VLV_SW: track 88.4 -> 0.00 mm
- net VCC: track 63.7 -> 0.00 mm
- net VLV1_SW: track 0.00 -> 63.6 mm
- net VLV2_SW: track 0.00 -> 48.6 mm
- net DISP_RST: track 0.00 -> 42.6 mm
- net LITE: track 12.2 -> 51.0 mm
- net SCL: track 24.3 -> 59.6 mm
- net GND: track 169.2 -> 134.4 mm
- net SCK: track 14.5 -> 49.0 mm
- net TE: track 0.00 -> 34.1 mm
- net CAN_ERR: track 32.0 -> 0.00 mm, vias 2 -> 0
- net CAN_RX: track 31.9 -> 0.00 mm
- net VLV1/2_SW_IO: track 0.00 -> 31.6 mm, vias 0 -> 2
- net VLV3/4_SW_IO: track 0.00 -> 31.6 mm
- net MOSI: track 15.6 -> 47.2 mm
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- added copper zone on layer 1, net 3.3V
- removed copper zone on layer 1, net VIN
Other:
- board size 78.7 x 113 mm -> 78.7 x 111.8 mm
- board text added: "3.3V"
- board text added: "DISP"
- board text added: "GND"
- board text added: "UPDI"
