File: eagle/printed/202403-zone_ctrl.sch (EAGLE design)
At the start: 95 parts, among them IC1 ATTINY426-MU, J10 1-770166-0, J11 1-770166-0, J13 FEMALE 2x3, J2 282834-8, J3 282834-8, J4 282834-8, J5 282834-8, J6 282834-8, J7 282834-8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

Commit message: Remove old eagle files now that we have git history
Parts:
- removed C8: 10nF, SparkFun-Capacitors:10NF-0603-50V-10%
- removed C9: 1.0uF, SparkFun-Capacitors:1.0UF-0603-16V-10%
- removed DL, VCC: PTR1B1,27, testpad:PTR1B1,27
- removed IC1: ATTINY426-MU, ATTINY426-MU:ATTINY426-MU
- removed J10: 1-770166-0, Terminals and sockets:1-770166-0
- removed J13: FEMALE 2x3, SparkFun-Connectors:CONN_03X2FEMALE
- removed Q2: 20V/4.2A/52mΩ/1.4W, SparkFun-DiscreteSemi:MOSFET_PCH-DMG2305UX-7
- removed R13, R14: 4.7k, SparkFun-Resistors:4.7KOHM-0603-1/10W-1%
- removed R17: 47k, SparkFun-Resistors:47KOHM-0603-1/10W-1%
- removed R3: 2.2k, SparkFun-Resistors:2.2KOHM-0603-1/10W-1%
- removed U3: MIC5504-3.3YM5-TR, MIC5504-3.3YM5-TR:MIC5504-3.3YM5-TR
- added BOOT, RST: JUMPER-SMT_2_NO_NO-SILK, SparkFun-Jumpers:JUMPER-SMT_2_NO_NO-SILK
- added BOOT_TP: PTR1B1,27, testpad:PTR1B1,27
- added D2, D3, D4, D5, D6: 1A/23V/620mV, SparkFun-DiscreteSemi:DIODE-SCHOTTKY-BAT20J
- added J12: 455-1750-1-ND, SparkFun-Connectors:CONN_03
- C1: device SparkFun-Capacitors:10UF-1210-50V-20% -> SparkFun-Capacitors:10UF-1206-6.3V-20%
- J9: value 282834-2 -> 282834-3; device TE terminal block 282834-2:282834-2 -> Terminals and sockets:282834-3
- L1: value 4.7μH -> 4.7μH_SHIELDED_INDUCTOR; device SparkFun-Coils:4.7μH_SHIELDED_INDUCTORNPIS_LS -> SparkFun-Coils:4.7μH_SHIELDED_INDUCTOR
- R1, R2: value 510 -> 2.2k; device Resistors:510OHM-0603-1/10W-5% -> SparkFun-Resistors:2.2KOHM-0603-1/10W-1%
- R20, R21, R22, R23, R24, R25, R26, R27, R28, R29, R30, R31, R32, R33, R34, R35: value 10k -> 22k; device SparkFun-Resistors:10KOHM-0603-1/10W-1% -> SparkFun-Resistors:22KOHM-0603-1/10W-1%
- R7, R8: value 4.7k -> 1k; device SparkFun-Resistors:4.7KOHM-0603-1/10W-1% -> SparkFun-Resistors:1KOHM-0603-1/10W-1%
- U1: value AP63205WU-7 -> AP63203WU-7; device Diodes buck converter:AP63205WU-7 -> Diodes buck converter:AP63203WU-7
- U2: value TJA1055T_3_2Z -> ATTINY426-MU; device TJA1055T_3_2Z:TJA1055T_3_2Z -> ATTINY426-MU:ATTINY426-MU
- X1: value JST-XH-04-PIN-ROUND-PAD -> JST-XH-02-PIN-ROUND-PAD; device Rembrandt Electronics - JST XH Connectors v1-0:JST-XH-04-PIN-ROUND-PAD -> Rembrandt Electronics - JST XH Connectors v1-0:JST-XH-02-PIN-ROUND-PAD
Connections:
- removed net CANH: R1.2, U2.CANH, X1-3.S
- removed net CANL: R2.2, U2.CANL, X1-2.S
- removed net CAN_ERR: R14.1, U2.!ERR, U4.IO8
- removed net CAN_RX: R13.1, U2.RXD, U4.IO17
- removed net CAN_TX: U2.TXD, U4.IO18
- removed net N$5: R2.1, U2.RTL
- removed net N$6: R1.1, U2.RTH
- removed net N$8: C8.2, R3.1, U2.!WAKE, U2.BAT
- removed net SD_CS: U4.IO13, X3.SD_CS
- removed net TS3_Y: J7.7, R34.2
- removed net TS3_Y_IO: IC1.PC1, U14.COLLECTOR_2
- removed net TS_CS: U4.IO14, X3.TS_CS
- removed net VCC: C3.1, C4.1, C5.1, L1.2, Q2.D, U1.FB, U2.!STB, U2.EN, U2.VCC, VCC.TP
- removed net VLV_SW: J2.4, J2.8, J3.4, J3.8, R32.2
- removed net VLV_SW_IO: IC1.PC3, U14.COLLECTOR_4
- new net DISP_RST: U4.IO12, X3.RESET
- new net TE: U4.IO3, X3.BUSY/TE
- new net VLV1/2_SW: D2.A, D5.C, R33.2
- new net VLV1/2_SW_IO: R2.1, U14.COLLECTOR_3, U2.PC2
- new net VLV1_SW: D2.C, J2.4
- new net VLV2_SW: D5.A, J2.8
- new net VLV3/4_SW: D3.C, D6.A, R32.2
- new net VLV3/4_SW_IO: R1.1, U14.COLLECTOR_4, U2.PC3
- new net VLV3_SW: D3.A, J3.4
- new net VLV4_SW: D6.C, J3.8
- net 3.3V: now also C3.1, C4.1, C5.2, J12.2, L1.2, R1.2, R2.2, U1.FB, U2.VDD; no longer IC1.VDD, J13.2, R13.2, R14.2, U3.VOUT
- net DC: now also U4.IO13; no longer U4.IO12
- net FC1_OB_IO: now also U2.(EXTCLK)_PA3; no longer IC1.(EXTCLK)_PA3
- net FC1_V_IO: now also U2.PA2; no longer IC1.PA2
- net FC2_OB_IO: now also U2.PA5; no longer IC1.PA5
- net FC2_V_IO: now also U2.PA4; no longer IC1.PA4
- net FC3_OB_IO: now also U2.PA7; no longer IC1.PA7
- net FC3_V_IO: now also U2.PA6; no longer IC1.PA6
- net FC4_OB_IO: now also U2.PB4; no longer IC1.PB4
- net FC4_V_IO: now also U2.PB5; no longer IC1.PB5
- net GND: now also BOOT.2, C5.1, J12.3, J9.3, RST.2, U2.EP, X1-2.S, X3.DISP_CS; no longer C5.2, C8.1, C9.1, IC1.EP, IC1.GND, J10.2, J13.6, R17.1, U3.GND, X1-4.S
- net LITE: now also U4.IO48; no longer U4.IO3
- net MISO: now also U4.IO14; no longer U4.IO11
- net MOSI: now also U4.IO21; no longer U4.IO10
- net N$3: now also BOOT.1, BOOT_TP.TP; no longer DL.TP
- net N$9: now also RST.1
- net REG_IN: now also C1.1, D4.C, U1.EN, U1.VIN; no longer C9.2, Q2.S, U3.EN, U3.VIN
- net SCK: now also U4.IO47; no longer U4.IO9
- net SCL: now also U4.IO11; no longer U4.IO21
- net SDA: now also U4.IO10; no longer U4.IO47
- net TS1_W_IO: now also U2.PB1; no longer IC1.PB1
- net TS1_Y_IO: now also U2.PB2_(TOSC2); no longer IC1.PB2_(TOSC2)
- net TS2_W_IO: now also U2.PB3_(TOSC1); no longer IC1.PB3_(TOSC1)
- net TS2_Y_IO: now also U2.PB0; no longer IC1.PB0
- net TS3_W_IO: now also U2.PC0; no longer IC1.PC0
- net TS4_W: now also R34.2; no longer R33.2
- net TS4_W_IO: now also U14.COLLECTOR_2, U2.PC1; no longer IC1.PC2, U14.COLLECTOR_3
- net TS_INT: now also U4.IO9; no longer U4.IO48
- net UART: now also U2.PA1; no longer IC1.PA1
- net UPDI: now also J12.1, U2.PA0_(UPDI/!RESET); no longer IC1.PA0_(UPDI/!RESET), J13.1
- net VIN: now also D4.A; no longer C1.1, J10.1, R3.2, U1.EN, U1.VIN
- net V_USB: no longer Q2.G, R17.2
Other:
- note added: "3.3V REGULATOR"
- note removed: "1uF filter on VOUT if not near other filters"
- note removed: "5V REGULATOR"
- note removed: "CAN INTERFACE"
- moved on the sheet: C5, D1, R1, R2, R40, U9, X1-1, X1-2
