File: eagle/rs485/zone_ctrl.brd (EAGLE design)
At the start: 78.7 x 111.8 mm, 91 parts, among them J11 1-770166-0, J12 455-1750-1-ND, J2 282834-8, J3 282834-8, J4 282834-8, J5 282834-8, J6 282834-8, J7 282834-8, J8 4DB-P108-04, J9 282834-3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

Commit message: start swapping A/B pins
Connections:
- net RS485A: now also J9.2, R40.2, U9.6; no longer J9.1, R40.1, U9.7
- net RS485B: now also J9.1, R40.1, U9.7; no longer J9.2, R40.2, U9.6
Routing:
- net RS485B: track 13.1 -> 9.45 mm
- net RS485A: track 9.45 -> 13.1 mm
Changed lines of the file:
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@@
 </layers>
 <board>
-<fusionsync huburn="a.cGVyc29uYWw6dWUyYTcxNGEx" projecturn="a.cGVyc29uYWw6dWUyYTcxNGExIzIwMjEwMjA5MzgwOTE4NjMx" f3durn="urn:adsk.wipprod:dm.lineage:DE_O0rDfRXSuypDpmkco8g" pcbguid="d01aefcd-c252-474d-beca-ed591bf99482" lastpulledtime="" lastsyncedchangeguid="" latestrevisionid="7dd453d7-232b-447a-bfce-c69fbf2cfd12" lastsyncedrevisionid="7dd453d7-232b-447a-bfce-c69fbf2cfd12" lastboardhashguid="4ea855a6-e991-f2e0-b084-2e673372e3e9" lastpushedtime="2024-06-22T03:14:57Z" linktopcb3d="true"/>
+<fusionsync huburn="a.cGVyc29uYWw6dWUyYTcxNGEx" projecturn="a.cGVyc29uYWw6dWUyYTcxNGExIzIwMjEwMjA5MzgwOTE4NjMx" f3durn="urn:adsk.wipprod:dm.lineage:DE_O0rDfRXSuypDpmkco8g" pcbguid="" lastpulledtime="" lastsyncedchangeguid="" latestrevisionid="7dd453d7-232b-447a-bfce-c69fbf2cfd12" lastsyncedrevisionid="7dd453d7-232b-447a-bfce-c69fbf2cfd12" lastboardhashguid="4ea855a6-e991-f2e0-b084-2e673372e3e9" lastpushedtime="2024-06-22T03:14:57Z" linktopcb3d="true"/>
 <plain>
 <wire x1="0" y1="0" x2="78.74" y2="0" width="0" layer="20"/>
@@
 <wire x1="72.517" y1="58.293" x2="40.005" y2="58.293" width="0.4064" layer="16"/>
 </signal>
-<signal name="RS485B">
+<signal name="RS485A">
 <contactref element="J9" pad="2"/>
 <contactref element="U9" pad="6"/>
@@
 <wire x1="10.541" y1="55.118" x2="11.43" y2="56.007" width="0.254" layer="1"/>
 </signal>
-<signal name="RS485A">
+<signal name="RS485B">
 <contactref element="U9" pad="7"/>
 <contactref element="J9" pad="1"/>
