File: eagle/rs485/zone_ctrl.sch (EAGLE design)
At the start: 91 parts, among them J11 1-770166-0, J12 455-1750-1-ND, J2 282834-8, J3 282834-8, J4 282834-8, J5 282834-8, J6 282834-8, J7 282834-8, J8 4DB-P108-04, J9 282834-3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

Commit message: start swapping A/B pins
Connections:
- net RS485A: now also J9.2, R40.2, U9.A; no longer J9.1, R40.1, U9.B
- net RS485B: now also J9.1, R40.1, U9.B; no longer J9.2, R40.2, U9.A
Changed lines of the file:
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@@
 </segment>
 </net>
-<net name="RS485B" class="0">
+<net name="RS485A" class="0">
 <segment>
 <label x="63.5" y="10.16" size="1.778" layer="95"/>
@@
 </segment>
 </net>
-<net name="RS485A" class="0">
+<net name="RS485B" class="0">
 <segment>
 <pinref part="U9" gate="G$1" pin="B"/>
