File: eagle/rs485/controller.brd (EAGLE design)
At the start: 51.3 x 58.8 mm, 48 parts, among them J2 282834-3, J4 JST-XH-04-PIN-ROUND-PAD, U1 AP63203WU-7, U2 SCD-40, U4 ESP32-S3-WROOM-1-N16R2, U5 G3VM-61VY3_TR_, U6 G3VM-61VY3_TR_, U7 RX8111CE_B0, U8 STS35-DIS, U9 SP3485CN-L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

Commit message: finish flipping RS485A/B
Connections:
- net RS485A: now also J4.3, JP1.1, U9.6; no longer J4.2, R40.1, U9.7
- net RS485B: now also J4.2, R40.1, U9.7; no longer J4.3, JP1.1, U9.6
Routing:
- net RS485B: track 25.1 -> 27.1 mm
- net RS485A: track 27.1 -> 25.1 mm
Changed lines of the file:
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@@
 <wire x1="18.315" y1="8.697" x2="18.415" y2="8.597" width="0.254" layer="1"/>
 </signal>
-<signal name="RS485B">
+<signal name="RS485A">
 <contactref element="U9" pad="6"/>
 <contactref element="J4" pad="3"/>
@@
 <wire x1="43.307" y1="4.572" x2="43.307" y2="3.429" width="0.254" layer="1"/>
 </signal>
-<signal name="RS485A">
+<signal name="RS485B">
 <contactref element="U9" pad="7"/>
 <contactref element="R40" pad="1"/>
