File: eagle/rs485/fancoil.brd (EAGLE design)
At the start: 38.1 x 30.5 mm, 23 parts, among them J1 1-770166-0, J13 FEMALE 2x3, J4 JST-XH-04-PIN-ROUND-PAD, Q1 600mA/40V, U1 AP63203WU-7, U2 LTV-814S, U3 ATTINY426-MU, U9 SP3485CN-L

Commit message: finish flipping RS485A/B
Connections:
- net RS485A: now also J4.3, JP1.1, U9.6; no longer J4.2, R40.1, U9.7
- net RS485B: now also J4.2, R40.1, U9.7; no longer J4.3, JP1.1, U9.6
Routing:
- net RS485B: track 27.1 -> 15.4 mm
- net RS485A: track 15.4 -> 27.1 mm
Changed lines of the file:
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@@
 <text x="4.318" y="17.907" size="1.778" layer="25">-</text>
 <text x="31.75" y="3.048" size="1.27" layer="25" rot="R180">VIN</text>
-<text x="31.75" y="5.588" size="1.27" layer="25" rot="R180">A</text>
-<text x="31.877" y="8.255" size="1.27" layer="25" rot="R180">B</text>
+<text x="31.75" y="5.588" size="1.27" layer="25" rot="R180">B</text>
+<text x="31.877" y="8.255" size="1.27" layer="25" rot="R180">A</text>
 <text x="31.877" y="10.795" size="1.27" layer="25" rot="R180">GND</text>
 <text x="4.953" y="30.099" size="0.6096" layer="25" rot="R180" align="bottom-right">SDA</text>
@@
 <wire x1="17.399" y1="24.511" x2="23.495" y2="18.415" width="0.254" layer="16"/>
 </signal>
-<signal name="RS485B">
+<signal name="RS485A">
 <contactref element="U9" pad="6"/>
 <contactref element="J4" pad="3"/>
@@
 <wire x1="36.83" y1="7.493" x2="35.687" y2="7.493" width="0.254" layer="1"/>
 </signal>
-<signal name="RS485A">
+<signal name="RS485B">
 <contactref element="U9" pad="7"/>
 <contactref element="R40" pad="1"/>
