File: eagle/rs485/fresh_air_control.brd (EAGLE design)
At the start: 53.3 x 47 mm, 39 parts, among them J13 FEMALE 2x3, J2 1-770166-0, J3 1-794073-0, J4 JST-XH-04-PIN-ROUND-PAD, Q1 200mA/40V, U1 AP63203WU-7, U2 ATTINY426-MU, U5 VO2223B-X007T, U6 TCMT1106, U7 TCMT1106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

Commit message: fresh air control updates
Parts:
- R8: value 4.7k -> 2.2k
- R9: value 4.7k -> 22k
Changed lines of the file:
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@@
 <attribute name="VALUE" value="10k" x="37.084" y="19.685" size="0.6096" layer="27" font="vector" ratio="20" rot="R180" align="top-center"/>
 </element>
-<element name="R8" library="SparkFun-Resistors" library_urn="urn:adsk.eagle:library:532" package="0603" package3d_urn="urn:adsk.eagle:package:41389018/1" value="4.7k" x="31.75" y="8.89" smashed="yes">
+<element name="R8" library="SparkFun-Resistors" library_urn="urn:adsk.eagle:library:532" package="0603" package3d_urn="urn:adsk.eagle:package:41389018/1" value="2.2k" x="31.75" y="8.89" smashed="yes">
 <attribute name="NAME" x="31.75" y="8.128" size="0.6096" layer="25" font="vector" ratio="20" rot="R180" align="bottom-center"/>
-<attribute name="PROD_ID" value="RES-07857" x="77.47" y="-41.91" size="1.778" layer="27" display="off"/>
-<attribute name="VALUE" value="4.7k" x="31.75" y="8.128" size="0.6096" layer="27" font="vector" ratio="20" align="top-center"/>
+<attribute name="PROD_ID" value="RES-08272" x="77.47" y="-41.91" size="1.778" layer="27" display="off"/>
+<attribute name="VALUE" value="2.2k" x="31.75" y="8.128" size="0.6096" layer="27" font="vector" ratio="20" align="top-center"/>
 </element>
-<element name="R9" library="SparkFun-Resistors" library_urn="urn:adsk.eagle:library:532" package="0603" package3d_urn="urn:adsk.eagle:package:41389018/1" value="4.7k" x="31.75" y="11.43" smashed="yes" rot="R180">
+<element name="R9" library="SparkFun-Resistors" library_urn="urn:adsk.eagle:library:532" package="0603" package3d_urn="urn:adsk.eagle:package:41389018/1" value="22k" x="31.75" y="11.43" smashed="yes" rot="R180">
 <attribute name="NAME" x="31.75" y="10.668" size="0.6096" layer="25" font="vector" ratio="20" rot="R180" align="bottom-center"/>
-<attribute name="PROD_ID" value="RES-07857" x="-17.78" y="62.23" size="1.778" layer="27" rot="R180" display="off"/>
-<attribute name="VALUE" value="4.7k" x="31.75" y="12.192" size="0.6096" layer="27" font="vector" ratio="20" rot="R180" align="top-center"/>
+<attribute name="PROD_ID" value="RES-07853" x="-17.78" y="62.23" size="1.778" layer="27" rot="R180" display="off"/>
+<attribute name="VALUE" value="22k" x="31.75" y="12.192" size="0.6096" layer="27" font="vector" ratio="20" rot="R180" align="top-center"/>
 </element>
 <element name="U1" library="Diodes buck converter" package="SOIC_05WU-7_DIO" value="AP63203WU-7" x="15.621" y="6.731" smashed="yes" rot="R90">

Commit message: finish flipping RS485A/B
Connections:
- net RS485A: now also J4.3, JP1.1, U9.6; no longer J4.2, R40.1, U9.7
- net RS485B: now also J4.2, R40.1, U9.7; no longer J4.3, JP1.1, U9.6
Routing:
- net RS485B: track 22.8 -> 18.8 mm
- net RS485A: track 18.8 -> 22.8 mm
Changed lines of the file:
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@@
 <wire x1="15.748" y1="33.02" x2="13.462" y2="33.02" width="0.254" layer="1"/>
 </signal>
-<signal name="RS485B">
+<signal name="RS485A">
 <contactref element="U9" pad="6"/>
 <contactref element="J4" pad="3"/>
@@
 <wire x1="21.336" y1="3.175" x2="20.8153" y2="3.6957" width="0.254" layer="1"/>
 </signal>
-<signal name="RS485A">
+<signal name="RS485B">
 <contactref element="U9" pad="7"/>
 <contactref element="R40" pad="1"/>
