File: eagle/rs485/fresh_air_control.sch (EAGLE design)
At the start: 39 parts, among them J13 FEMALE 2x3, J2 1-770166-0, J3 1-794073-0, J4 JST-XH-04-PIN-ROUND-PAD, Q1 200mA/40V, U1 AP63203WU-7, U2 ATTINY426-MU, U5 VO2223B-X007T, U6 TCMT1106, U7 TCMT1106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

Commit message: fresh air control updates
Parts:
- R8: value 4.7k -> 2.2k; device SparkFun-Resistors:4.7KOHM-0603-1/10W-1% -> SparkFun-Resistors:2.2KOHM-0603-1/10W-1%
- R9: value 4.7k -> 22k; device SparkFun-Resistors:4.7KOHM-0603-1/10W-1% -> SparkFun-Resistors:22KOHM-0603-1/10W-1%
Other:
- note added: "consider pull R8 high to M+15 make R8/9 4.7k"
- note removed: "consider pull R8 high to M+15 switching R9 to 2.2k (or R8 too)"
Changed lines of the file:
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@@
 <part name="GND7" library="SparkFun-PowerSymbols" library_urn="urn:adsk.eagle:library:530" deviceset="GND" device=""/>
 <part name="Q1" library="SparkFun-DiscreteSemi" library_urn="urn:adsk.eagle:library:514" deviceset="TRANS_PNP" device="-PMBT3906|MMBT3906L" package3d_urn="urn:adsk.eagle:package:38446/2" value="200mA/40V"/>
-<part name="R8" library="SparkFun-Resistors" library_urn="urn:adsk.eagle:library:532" deviceset="4.7KOHM" device="-0603-1/10W-1%" package3d_urn="urn:adsk.eagle:package:41389018/1" value="4.7k"/>
-<part name="R9" library="SparkFun-Resistors" library_urn="urn:adsk.eagle:library:532" deviceset="4.7KOHM" device="-0603-1/10W-1%" package3d_urn="urn:adsk.eagle:package:41389018/1" value="4.7k"/>
+<part name="R8" library="SparkFun-Resistors" library_urn="urn:adsk.eagle:library:532" deviceset="2.2KOHM" device="-0603-1/10W-1%" package3d_urn="urn:adsk.eagle:package:41389018/1" value="2.2k"/>
+<part name="R9" library="SparkFun-Resistors" library_urn="urn:adsk.eagle:library:532" deviceset="22KOHM" device="-0603-1/10W-1%" package3d_urn="urn:adsk.eagle:package:41389018/1" value="22k"/>
 <part name="R10" library="Resistors" deviceset="120OHM" device="-0603-1/10W-5%" package3d_urn="urn:adsk.eagle:package:41389018/1" value="120"/>
 <part name="R5" library="SparkFun-Resistors" library_urn="urn:adsk.eagle:library:532" deviceset="2.2KOHM" device="-0603-1/10W-1%" package3d_urn="urn:adsk.eagle:package:41389018/1" value="2.2k"/>
@@
 <text x="184.404" y="27.432" size="1.778" layer="94">MOTOR POWER</text>
 <text x="292.1" y="43.18" size="1.778" layer="94" rot="R90">consider pull R8 high to M+15
-switching R9 to 2.2k (or R8 too)</text>
+make R8/9 4.7k</text>
 </plain>
 <instances>

Commit message: finish flipping RS485A/B
Connections:
- net RS485A: now also J4-3.S, JP1.1, U9.A; no longer J4-2.S, R40.1, U9.B
- net RS485B: now also J4-2.S, R40.1, U9.B; no longer J4-3.S, JP1.1, U9.A
Changed lines of the file:
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@@
 </segment>
 </net>
-<net name="RS485B" class="0">
+<net name="RS485A" class="0">
 <segment>
 <label x="40.64" y="27.94" size="1.778" layer="95"/>
@@
 </segment>
 </net>
-<net name="RS485A" class="0">
+<net name="RS485B" class="0">
 <segment>
 <wire x1="40.64" y1="30.48" x2="66.04" y2="30.48" width="0.1524" layer="91"/>
